File: kicad/possu2.kicad_pcb (KiCad board)
At the start: 2 copper layers, 45 parts, among them IC1 ATTINY861-S, P1 CONN_6, P2 CONN_2, SW1 SW_PUSH

Commit message: Piirsin salamaan edgecutsit ja tein valmistusgerberit jotta voidaan tilata
Other:
- board outline added: 48.9 x 67.3 mm
